File: HARDWARE-DESIGN/OSMAN - REV3.0/Mergen Ground Station_V2.0.sch (EAGLE design)
At the start: 70 parts, among them J2 CON-SD-CARD_MICROSD-2908-05, J4 U.FL, U1 STM32F302C8T6, U13 L86, U15 AMS1117-5V, U16 AMS1117-3.3, X2 JST-XH-04-PIN-LONG-PAD, Y1 ABMM2-8.000MHZ-E2-T

Commit message: Version 3.0 was relased by brain.dll
Parts:
- removed SG2: F/CM12P, buzzer:F/CM12P
- removed U1: STM32F302C8T6, STM32F302C8T6:STM32F302C8T6
- added D2: GREEN, SparkFun-LED:LED0603
- added LS1: CMT-8530S-SMT, SMT-BUZZER:CMT-8530S-SMT
- added R2: 10k, rcl:R-EU_R0603
- added R3: 1.5k, rcl:R-EU_R0603
- added U2: (no value), STM32F103C8T6:STM32F103C8T6
- added VBAT_D: 3.3k, SparkFun-Resistors:2.0KOHM1/10W5%(0603)
- added VBAT_U: 10k, SparkFun-Resistors:2.0KOHM1/10W5%(0603)
Connections:
- removed net INT: U1A.PC13-WKUP2
- removed net N$28: R32.2, SG2.1
- removed net USB_D+: J5.D+, U1A.PA12
- removed net USB_D-: J5.D-, U1A.PA11
- new net LED2: D2.A, U2A.PA7
- new net N$3: D2.C, R3.2
- new net N$4: LS1.P, R32.2
- new net USB_N: J5.D-, U2A.PA11
- new net USB_P: J5.D+, U2A.PA12
- new net VB: U2A.PA6, VBAT_D.2, VBAT_U.1
- net 3.3V: now also U2B.VBAT, U2B.VDD_1, U2B.VDD_2, U2B.VDD_3; no longer U1B.VBAT, U1B.VDD_1, U1B.VDD_2, U1B.VDD_3
- net AUX: now also U2A.PA5; no longer U1A.PA4
- net BT0: now also U2A.BOOT0; no longer U1A.BOOT0
- net BZZR: now also U2A.PB4; no longer U1A.PA7
- net CS: now also U2A.PB12; no longer U1A.PA8
- net DRDY: now also R2.2, U2A.PB5
- net FN: now also U2A.PA8; no longer U1A.PB5
- net GND: now also LS1.N, R2.1, R3.1, U2B.VSSA, U2B.VSS_1, U2B.VSS_2, U2B.VSS_3, VBAT_D.1; no longer SG2.2, U1B.VSSA/VREF-, U1B.VSS_1, U1B.VSS_2, U1B.VSS_3
- net LED: now also U2A.PB0; no longer U1A.PB0
- net M0: now also U2A.PA0-WKUP; no longer U1A.PA0-WKUP1
- net M1: now also U2A.PA1; no longer U1A.PA1
- net MISO: now also U2A.PB14; no longer U1A.PB14
- net MOSI: now also U2A.PB15; no longer U1A.PB15
- net NRST: now also U2A.NRST; no longer U1A.NRST
- net OSC_IN: now also U2A.OSC_IN; no longer U1A.PF0-OSC_IN
- net OSC_OUT: now also U2A.OSC_OUT; no longer U1A.PF1-OSC_OUT
- net RX1: now also U2A.PA10; no longer U1A.PB7
- net RX2: now also U2A.PA3; no longer U1A.PA3
- net RX3: now also U2A.PB11; no longer U1A.PB11
- net SCK: now also U2A.PB13; no longer U1A.PB3
- net SCL: now also U2A.PB6; no longer U1A.PA9
- net SDA: now also U2A.PB7; no longer U1A.PA10
- net SWCLK: now also U2A.PA14; no longer U1A.PA14
- net SWDIO: now also U2A.PA13; no longer U1A.PA13
- net TX1: now also U2A.PA9; no longer U1A.PB6
- net TX2: now also U2A.PA2; no longer U1A.PA2
- net TX3: now also U2A.PB10; no longer U1A.PB10
- net VCC: now also VBAT_U.2
- net VDDA: now also U2B.VDDA; no longer U1B.VDDA/VREF+
Other:
- note added: "8M-CRYSTAL"
- note added: "BATTARY VOLTAGE"
- note added: "BOOT AND RESET"
- note added: "LDO 3.3V"
- note added: "LDO 5V"
- note added: "MAGNETOMETER"
- note added: "MARKERS"
- note added: "MCU"
- note added: "POWER SUPPLY"
- note added: "SD CARD SLOT"
- note added: "UART SOCKET"
- note added: "USB SOCKET"
- note removed: "Mergen Ground Station"
