File: HARDWARE-DESIGN/REV3.0/Mergen Ground Station_V2.0.sch (EAGLE design)
At the start: 75 parts, among them J2 CON-SD-CARD_MICROSD-2908-05, J4 U.FL, U13 L86, U15 AMS1117-5V, U16 AMS1117-3.3, X2 JST-XH-04-PIN-LONG-PAD, Y1 ABMM2-8.000MHZ-E2-T

Commit message: new buzzer was added
Parts:
- removed LS1: CMT-8530S-SMT, SMT-BUZZER:CMT-8530S-SMT
- added LS2: CMT-7525S-SMT, CMT-7525S-SMT:CMT-7525S-SMT
Connections:
- net GND: now also LS2.N; no longer LS1.N
- net N$4: now also LS2.P; no longer LS1.P
Changed lines of the file:
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@@
 <part name="R3" library="rcl" library_urn="urn:adsk.eagle:library:334" deviceset="R-EU_" device="R0603" package3d_urn="urn:adsk.eagle:package:23555/3" value="1.5k"/>
 <part name="GND12" library="supply1" library_urn="urn:adsk.eagle:library:371" deviceset="GND" device=""/>
-<part name="LS1" library="SMT-BUZZER" deviceset="CMT-8530S-SMT" device=""/>
+<part name="LS2" library="CMT-7525S-SMT" deviceset="CMT-7525S-SMT" device=""/>
 </parts>
 <sheets>
@@
 <attribute name="VALUE" x="254" y="26.67" size="1.778" layer="96" rot="R90"/>
 </instance>
-<instance part="LS1" gate="G$1" x="246.38" y="50.8" smashed="yes" rot="R90">
-<attribute name="NAME" x="237.482090625" y="46.986609375" size="1.77958125" layer="95" rot="R90"/>
-<attribute name="VALUE" x="257.8248" y="46.985059375" size="1.780309375" layer="96" rot="R90"/>
+<instance part="LS2" gate="G$1" x="246.38" y="50.8" smashed="yes" rot="R90">
+<attribute name="NAME" x="237.488159375" y="46.989209375" size="1.77836875" layer="95" rot="R90"/>
+<attribute name="VALUE" x="257.8274" y="46.98418125" size="1.780709375" layer="96" rot="R90"/>
 </instance>
 </instances>
@@
 </segment>
 <segment>
-<pinref part="LS1" gate="G$1" pin="N"/>
 <pinref part="GND49" gate="1" pin="GND"/>
 <wire x1="251.46" y1="50.8" x2="255.27" y2="50.8" width="0.1524" layer="91"/>
+<pinref part="LS2" gate="G$1" pin="N"/>
 </segment>
 </net>
@@
 <segment>
 <pinref part="R32" gate="G$1" pin="2"/>
-<pinref part="LS1" gate="G$1" pin="P"/>
 <wire x1="236.22" y1="50.8" x2="241.3" y2="50.8" width="0.1524" layer="91"/>
-</segment>
-</net>
+<pinref part="LS2" gate="G$1" pin="P"/>
+</segment>
+</net>
